Commit message: got wheels to align with robot

File: p2/catkin_ws/src/my_robot/urdf/my_robot.xacro (robot description, xacro)
@@ -35,5 +35,5 @@
     <inertial>
       <mass value="5.0"/>
-      <origin xyz="0 -0.3 0" rpy=" 0 1.5707 1.5707"/>
+      <origin xyz="0 -0.1 0" rpy=" 0 1.5707 1.5707"/>
       <inertia
           ixx="0.1" ixy="0" ixz="0"
@@ -43,5 +43,5 @@
     </inertial>
     <collision name='collision'>
-      <origin xyz="0 -0.3 0" rpy=" 0 1.5707 1.5707"/>
+      <origin xyz="0 -0.1 0" rpy=" 0 1.5707 1.5707"/>
       <geometry>
         <cylinder radius="0.1" length="0.05"/>
@@ -49,5 +49,5 @@
     </collision>
     <visual name='R_wheel_visual'>
-      <origin xyz="0 -0.3 0" rpy=" 0 1.5707 1.5707"/>
+      <origin xyz="0 -0.1 0" rpy=" 0 1.5707 1.5707"/>
       <geometry>
         <cylinder radius="0.1" length="0.05"/>
@@ -112,8 +112,8 @@
   </joint>
   <joint type="continuous" name="R_wheel_hinge">
-   <origin xyz="0 -0.3 0" rpy="0 0 0"/>
+   <origin xyz="0 -0.1 0" rpy="0 0 0"/>
    <child link="R_wheel"/>
    <parent link="chassis"/>
-   <axis xyz="0 -0.3 0" rpy="0 0 0"/>
+   <axis xyz="0 -0.1 0" rpy="0 0 0"/>
    <limit effort="10000" velocity="1000"/>
    <dynamics damping="1.0" friction="1.0"/>

Commit message: added lidar

File: p2/catkin_ws/src/my_robot/urdf/my_robot.xacro (robot description, xacro)
@@ -103,4 +103,56 @@
     </visual>
   </link>
+ <joint name="camera_joint" type="fixed">
+    <axis xyz="0 1 0" />
+    <origin xyz="0.2 0 0" rpy="0 0 0"/>
+    <parent link="chassis"/>
+    <child link="camera"/>
+  </joint>
+  <link name="camera">
+    <collision>
+      <origin xyz="0.2 0 0" rpy="0 0 0"/>
+      <geometry>
+    	<box size=".05 .05 .05"/>
+      </geometry>
+    </collision>
+    <visual>
+      <origin xyz="0 0 0" rpy="0 0 0"/>
+      <geometry>
+   <box size=".05 .05 .05"/>
+      </geometry>
+      <material name="red"/>
+    </visual>
+    <inertial>
+      <mass value="0.1" />
+      <origin xyz="0 0 0" rpy="0 0 0"/>
+      <box_inertia m="0.1" x="0.05" y="0.05" z="0.05" />
+      <inertia ixx="1e-6" ixy="0" ixz="0" iyy="1e-6" iyz="0" izz="1e-6" />
+    </inertial>
+  </link>
+ <joint name="hokuyo_joint" type="fixed">
+    <axis xyz="0 1 0" />
+    <origin xyz="0.15 0 0.08" rpy="0 0 0"/>
+    <parent link="chassis"/>
+    <child link="hokuyo"/>
+  </joint>
+  <link name="hokuyo">
+    <collision>
+      <origin xyz="0 0 0" rpy="0 0 0"/>
+      <geometry>
+    	<box size="0.1 0.1 0.1"/>
+      </geometry>
+    </collision>
+    <visual>
+      <origin xyz="0 0 0" rpy="0 0 0"/>
+      <geometry>
+   <mesh filename="package://my_robot/meshes/hokuyo.dae"/>
+      </geometry>
+    </visual>
+    <inertial>
+      <mass value="1e-5" />
+      <origin xyz="0 0 0" rpy="0 0 0"/>
+      <inertia ixx="1e-6" ixy="0" ixz="0" iyy="1e-6" iyz="0" izz="1e-6" />
+    </inertial>
+  </link>
   <joint type="continuous" name="L_wheel_hinge">
    <origin xyz="0 0.15 0" rpy="0 0 0"/>
@@ -112,8 +164,8 @@
   </joint>
   <joint type="continuous" name="R_wheel_hinge">
-   <origin xyz="0 -0.1 0" rpy="0 0 0"/>
+   <origin xyz="0 -0.07 0" rpy="0 0 0"/>
    <child link="R_wheel"/>
    <parent link="chassis"/>
-   <axis xyz="0 -0.1 0" rpy="0 0 0"/>
+   <axis xyz="0 -0.07 0" rpy="0 0 0"/>
    <limit effort="10000" velocity="1000"/>
    <dynamics damping="1.0" friction="1.0"/>

Commit message: trying to run simulator but odom isnt showing up

File: p2/catkin_ws/src/my_robot/urdf/my_robot.xacro (robot description, xacro)
@@ -1,4 +1,5 @@
 <?xml version='1.0'?>
 <robot name="my_robot" xmlns:xacro="http://www.ros.org/wiki/xacro">
+  <xacro:include filename="$(find my_robot)/urdf/my_robot.gazebo" />
   <link name="robot_footprint"></link>
   <joint name="robot_footprint_joint" type="fixed">
@@ -103,10 +104,4 @@
     </visual>
   </link>
- <joint name="camera_joint" type="fixed">
-    <axis xyz="0 1 0" />
-    <origin xyz="0.2 0 0" rpy="0 0 0"/>
-    <parent link="chassis"/>
-    <child link="camera"/>
-  </joint>
   <link name="camera">
     <collision>
@@ -130,10 +125,4 @@
     </inertial>
   </link>
- <joint name="hokuyo_joint" type="fixed">
-    <axis xyz="0 1 0" />
-    <origin xyz="0.15 0 0.08" rpy="0 0 0"/>
-    <parent link="chassis"/>
-    <child link="hokuyo"/>
-  </joint>
   <link name="hokuyo">
     <collision>
@@ -155,4 +144,16 @@
     </inertial>
   </link>
+ <joint name="camera_joint" type="fixed">
+    <axis xyz="0 1 0" />
+    <origin xyz="0.2 0 0" rpy="0 0 0"/>
+    <parent link="chassis"/>
+    <child link="camera"/>
+  </joint>
+ <joint name="hokuyo_joint" type="fixed">
+    <axis xyz="0 1 0" />
+    <origin xyz="0.15 0 0.08" rpy="0 0 0"/>
+    <parent link="chassis"/>
+    <child link="hokuyo"/>
+  </joint>
   <joint type="continuous" name="L_wheel_hinge">
    <origin xyz="0 0.15 0" rpy="0 0 0"/>
@@ -164,8 +165,8 @@
   </joint>
   <joint type="continuous" name="R_wheel_hinge">
-   <origin xyz="0 -0.07 0" rpy="0 0 0"/>
+   <origin xyz="0 -0.1 0" rpy="0 0 0"/>
    <child link="R_wheel"/>
    <parent link="chassis"/>
-   <axis xyz="0 -0.07 0" rpy="0 0 0"/>
+   <axis xyz="0 -0.5 0" rpy="0 0 0"/>
    <limit effort="10000" velocity="1000"/>
    <dynamics damping="1.0" friction="1.0"/>

Commit message: robot moves in riv

File: p2/catkin_ws/src/my_robot/urdf/my_robot.xacro (robot description, xacro)
@@ -168,5 +168,5 @@
    <child link="R_wheel"/>
    <parent link="chassis"/>
-   <axis xyz="0 -0.5 0" rpy="0 0 0"/>
+   <axis xyz="0 -0.25 0" rpy="0 0 0"/>
    <limit effort="10000" velocity="1000"/>
    <dynamics damping="1.0" friction="1.0"/>

Commit message: robot chases after ball

File: p2/catkin_ws/src/my_robot/urdf/my_robot.xacro (robot description, xacro)
@@ -36,5 +36,5 @@
     <inertial>
       <mass value="5.0"/>
-      <origin xyz="0 -0.1 0" rpy=" 0 1.5707 1.5707"/>
+      <origin xyz="0 0 0" rpy=" 0 1.5707 1.5707"/>
       <inertia
           ixx="0.1" ixy="0" ixz="0"
@@ -44,5 +44,5 @@
     </inertial>
     <collision name='collision'>
-      <origin xyz="0 -0.1 0" rpy=" 0 1.5707 1.5707"/>
+      <origin xyz="0 0 0" rpy=" 0 1.5707 1.5707"/>
       <geometry>
         <cylinder radius="0.1" length="0.05"/>
@@ -50,8 +50,11 @@
     </collision>
     <visual name='R_wheel_visual'>
-      <origin xyz="0 -0.1 0" rpy=" 0 1.5707 1.5707"/>
+      <origin xyz="0 0 0" rpy=" 0 1.5707 1.5707"/>
       <geometry>
         <cylinder radius="0.1" length="0.05"/>
       </geometry>
+	<material name="color1">
+		<color rgba="1 1 1 1"/>
+	</material>
     </visual>
   </link>
@@ -165,8 +168,8 @@
   </joint>
   <joint type="continuous" name="R_wheel_hinge">
-   <origin xyz="0 -0.1 0" rpy="0 0 0"/>
+   <origin xyz="0 -0.15 0" rpy="0 0 0"/>
    <child link="R_wheel"/>
    <parent link="chassis"/>
-   <axis xyz="0 -0.25 0" rpy="0 0 0"/>
+   <axis xyz="0 1 0" rpy="0 0 0"/>
    <limit effort="10000" velocity="1000"/>
    <dynamics damping="1.0" friction="1.0"/>
